File: digital/kicad/_autosave-digital_kicad.kicad_sch (KiCad schematic)
At the start: 16 parts, among them J1 Barrel_Jack_Switch, J2 Screw_Terminal_01x02, Q1 2N3904, Q2 2N3904, Q4 2N3904, SW1 SW_SPST

Commit message: kicad + pcb scheme review
Parts:
- added R7: 33k, Resistor_SMD:R_0805_2012Metric_Pad1.20x1.40mm_HandSolder, symbol Device:R
- A1: footprint Module:Arduino_Nano -> PCM_arduino-library:Arduino_Nano_Socket
- J1: footprint (none) -> Connector_BarrelJack:BarrelJack_Wuerth_6941xx301002
- J2: footprint (none) -> TerminalBlock_Phoenix:TerminalBlock_Phoenix_MKDS-1,5-2-5.08_1x02_P5.08mm_Horizontal
Connections:
- net +5V: no longer J1.2, J1.3
- net GND: now also J1.2, J1.3, R7.1
- net at J2.1 (Pin_1), R4.2: now also R7.2
- net VDC: now reaches A1.VIN, J1.1
Other:
- moved on the sheet: J1
