File: digital/kicad/digital_kicad.kicad_pcb (KiCad board)
At the start: 2 copper layers, 48.3 x 20.3 mm, 25 parts, among them J1 Conn_01x01_Pin, J2 Conn_01x01_Pin, J3 Conn_01x01_Pin, J4 Conn_01x01_Pin, Q1 2N3904, Q2 2N3904, Q3 FDN340P, Q4 2N3904, SW1 SW_SPST

Commit message: sync latest adjustments for final presentation
Other:
- outline, holes or cut-outs redrawn
Changed lines of the file:
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@@
 			(sketchdnponfab yes)
 			(crossoutdnponfab yes)
-			(subtractmaskfromsilk no)
+			(subtractmaskfromsilk yes)
 			(outputformat 1)
 			(mirror no)
 			(drillshape 0)
 			(scaleselection 1)
-			(outputdirectory "digital_v1")
+			(outputdirectory "../Gerber/")
 		)
 	)
@@
 	)
 	(gr_line
-		(start 111.76 66.04)
-		(end 154.94 66.04)
+		(start 109.22 66.04)
+		(end 157.48 66.04)
 		(stroke
 			(width 0.05)
@@
 	)
 	(gr_line
-		(start 157.48 63.5)
-		(end 157.48 48.26)
-		(stroke
-			(width 0.05)
-			(type default)
-		)
-		(layer "Edge.Cuts")
-	)
-	(gr_arc
-		(start 109.22 48.26)
-		(mid 109.963949 46.463949)
-		(end 111.76 45.72)
-		(stroke
-			(width 0.05)
-			(type default)
-		)
-		(layer "Edge.Cuts")
-	)
-	(gr_arc
-		(start 111.76 66.04)
-		(mid 109.963949 65.296051)
-		(end 109.22 63.5)
+		(start 157.48 66.04)
+		(end 157.48 45.72)
 		(stroke
 			(width 0.05)
@@
 	)
 	(gr_line
-		(start 154.94 45.72)
-		(end 111.76 45.72)
+		(start 157.48 45.72)
+		(end 109.22 45.72)
 		(stroke
 			(width 0.05)
@@
 	)
 	(gr_line
-		(start 109.22 48.26)
-		(end 109.22 63.5)
-		(stroke
-			(width 0.05)
-			(type default)
-		)
-		(layer "Edge.Cuts")
-	)
-	(gr_arc
-		(start 154.94 45.72)
-		(mid 156.736051 46.463949)
-		(end 157.48 48.26)
-		(stroke
-			(width 0.05)
-			(type default)
-		)
-		(layer "Edge.Cuts")
-	)
-	(gr_arc
-		(start 157.48 63.5)
-		(mid 156.736051 65.296051)
-		(end 154.94 66.04)
+		(start 109.22 45.72)
+		(end 109.22 66.04)
 		(stroke
 			(width 0.05)
@@
 		(polygon
 			(pts
-				(xy 110.053289 46.732561) (xy 156.562618 46.732561) (xy 156.562618 65.05572) (xy 110.053289 65.05572)
+				(xy 109.337347 45.825552) (xy 157.321453 45.825552) (xy 157.321453 66.04) (xy 109.337347 66.04)
 			)
 		)
