File: analog/kicad/scheme.kicad_sch (KiCad schematic)
At the start: 17 parts, among them U1 LM324

Commit message: restructuring analog
Parts:
- removed D2, D3, D4: NSCW100, symbol ltspice:LED
- added D2, D3, D4: LED, symbol Device:LED
- U1: value LM324 -> LM324N; footprint (none) -> Package_DIP:DIP-14_W7.62mm
Connections:
- net GND: now also D1.1 (K), D2.1 (K), D3.1 (K), D4.1 (K); no longer U1.13 (-)
- net OUT: now also U1.10 (+), U1.5 (+); no longer U1.6 (-), U1.9 (-)
- net VCC: no longer D1.2 (A)
- net dist2: now also U1.9 (-); no longer U1.10 (+)
- net dist3: now also U1.12 (+), U1.6 (-); no longer U1.5 (+)
- net at C1.1, R1.1, U1.2 (-): now also D1.2 (A); no longer D1.1 (K)
- net at R8.1: now also D3.2 (A)
- net at R7.1: now also D2.2 (A)
- net at R9.1: now also D4.2 (A)
- net at U1.14: now also U1.13 (-); no longer U1.12 (+)
Other:
- note removed: "BPW34"
- moved on the sheet: C1, R1

Commit message: kicad pcb and other fixes
Parts:
- removed C1: 22p, symbol ltspice:cap
- removed C2: 1µ, symbol ltspice:cap
- removed R1: 500k, symbol ltspice:res
- removed R2, R7, R8, R9: 220, symbol ltspice:res
- removed R3, R6: 10k, symbol ltspice:res
- removed R4: 14.7k, symbol ltspice:res
- removed R5: 5k, symbol ltspice:res
- removed V1: 5V, symbol ltspice:voltage
- added C1: 22p, Capacitor_SMD:C_0603_1608Metric, symbol Device:C_Small
- added C2: 1u, Capacitor_SMD:C_0603_1608Metric, symbol Device:C_Small
- added J1: Barrel_Jack_Switch, Connector_BarrelJack:BarrelJack_GCT_DCJ200-10-A_Horizontal, symbol Connector:Barrel_Jack_Switch
- added R1: 500k, Resistor_SMD:R_0603_1608Metric, symbol Device:R
- added R2: 220, Resistor_SMD:R_0603_1608Metric, symbol Device:R
- added R3, R6: 10k, Resistor_SMD:R_0603_1608Metric, symbol Device:R
- added R4: 14.7k, Resistor_SMD:R_0603_1608Metric, symbol Device:R
- added R5: 5k, Resistor_SMD:R_0603_1608Metric, symbol Device:R
- added R7, R8, R9: 1k, Resistor_SMD:R_0603_1608Metric, symbol Device:R
- D2, D3, D4: footprint (none) -> LED_THT:LED_D5.0mm
- U1: value LM324N -> LM324; footprint Package_DIP:DIP-14_W7.62mm -> Package_DIP:DIP-14_W7.62mm_Socket
Connections:
- net BIAS: now also C2.2, R2.2, R3.1
- net GND: now also C2.1, J1.2, R2.1, R6.1
- net OUT: now also C1.2, R1.2
- net dist2: now also R5.1, R6.2
- net dist3: now also R4.2, R5.2
- net at D1.2 (A), U1.2 (-): now also C1.1, R1.1
- net at D3.2 (A): now also R8.2
- net at U1.8: now also R8.1
- net at D4.2 (A): now also R9.2
- net at D2.2 (A): now also R7.2
- net at U1.7: now also R7.1
- net VCC: no longer names the net of U1.4 (V+)
- net VCC: now also J1.1, R3.2, R4.1, R9.1
- no-connect marks 0 -> 1
Other:
- moved on the sheet: D1, D2, D3, D4, U1A, U1B, U1C, U1D, U1E

Commit message: schematic in 9V out 5V
Parts:
- added R?: 12.5k, symbol Device:R
- added R?: 10k, symbol Device:R
Connections:
- net GND: now also R?.2
- net at R3.2, R4.1, R9.1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: now also R?.1, R?.2; no longer J1.1
- new net: J1.1, R?.1
Other:
- moved on the sheet: J1
Changed lines of the file:
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@@
 	(paper "A4")
+	(junction
+		(at 109.22 72.39)
+		(diameter 0)
+		(color 0 0 0 0)
+	)
 	(junction
 		(at 116.84 96.52)
@@
 	)
 	(junction
-		(at 116.84 72.39)
-		(diameter 0)
-		(color 0 0 0 0)
-	)
-	(junction
 		(at 132.08 113.03)
 		(diameter 0)
@@
 	)
 	(junction
+		(at 116.84 72.39)
+		(diameter 0)
+		(color 0 0 0 0)
+	)
+	(junction
 		(at 186.69 113.03)
 		(diameter 0)
@@
 	)
 	(junction
+		(at 99.06 77.47)
+		(diameter 0)
+		(color 0 0 0 0)
+	)
+	(junction
 		(at 139.7 99.06)
 		(diameter 0)
@@
 	)
 	(no_connect
-		(at 111.76 74.93)
+		(at 99.06 74.93)
 	)
 	(wire
@@
 	(wire
 		(pts
+			(xy 109.22 72.39) (xy 116.84 72.39)
+		)
+		(stroke
+			(width 0)
+			(type default)
+		)
+	)
+	(wire
+		(pts
 			(xy 113.03 102.87) (xy 111.76 102.87)
 		)
@@
 	(wire
 		(pts
+			(xy 109.22 72.39) (xy 109.22 73.66)
+		)
+		(stroke
+			(width 0)
+			(type default)
+		)
+	)
+	(wire
+		(pts
 			(xy 139.7 100.33) (xy 139.7 99.06)
 		)
@@
 	(wire
 		(pts
-			(xy 111.76 72.39) (xy 116.84 72.39)
-		)
-		(stroke
-			(width 0.1524)
-			(type solid)
+			(xy 99.06 85.09) (xy 109.22 85.09)
+		)
+		(stroke
+			(width 0)
+			(type default)
 		)
 	)
@@
 	(wire
 		(pts
+			(xy 106.68 72.39) (xy 109.22 72.39)
+		)
+		(stroke
+			(width 0)
+			(type default)
+		)
+	)
+	(wire
+		(pts
 			(xy 116.84 72.39) (xy 139.7 72.39)
 		)
@@
 	(wire
 		(pts
+			(xy 109.22 85.09) (xy 109.22 81.28)
+		)
+		(stroke
+			(width 0)
+			(type default)
+		)
+	)
+	(wire
+		(pts
 			(xy 186.69 113.03) (xy 186.69 120.65)
 		)
@@
 	(wire
 		(pts
+			(xy 99.06 77.47) (xy 102.87 77.47)
+		)
+		(stroke
+			(width 0)
+			(type default)
+		)
+	)
+	(wire
+		(pts
 			(xy 149.86 104.14) (xy 152.4 104.14)
 		)
@@
 		(pts
 			(xy 167.64 123.19) (xy 167.64 129.54)
+		)
+		(stroke
+			(width 0)
+			(type default)
+		)
+	)
+	(wire
+		(pts
+			(xy 99.06 77.47) (xy 99.06 85.09)
 		)
 		(stroke
@@
 	(symbol
 		(lib_id "power:GND")
-		(at 111.76 77.47 0)
+		(at 102.87 77.47 0)
 		(unit 1)
 		(exclude_from_sim no)
@@
 		(fields_autoplaced yes)
 		(property "Reference" "#PWR06"
-			(at 111.76 83.82 0)
+			(at 102.87 83.82 0)
 			(effects
 				(font
@@
 		)
 		(property "Value" "GND"
-			(at 111.76 82.55 0)
+			(at 102.87 82.55 0)
 			(effects
 				(font
@@
 		)
 		(property "Footprint" ""
-			(at 111.76 77.47 0)
+			(at 102.87 77.47 0)
 			(effects
 				(font
@@
 		)
 		(property "Datasheet" ""
-			(at 111.76 77.47 0)
+			(at 102.87 77.47 0)
 			(effects
 				(font
@@
 		)
 		(property "Description" "Power symbol creates a global label with name \"GND\" , ground"
-			(at 111.76 77.47 0)
+			(at 102.87 77.47 0)
 			(effects
 				(font
@@
 	)
 	(symbol
+		(lib_id "Device:R")
+		(at 109.22 77.47 0)
+		(unit 1)
+		(exclude_from_sim no)
+		(in_bom yes)
+		(on_board yes)
+		(dnp no)
+		(fields_autoplaced yes)
+		(property "Reference" "R?"
+			(at 111.76 76.1999 0)
+			(effects
+				(font
+					(size 1.27 1.27)
+				)
+				(justify left)
+			)
+		)
+		(property "Value" "12.5k"
+			(at 111.76 78.7399 0)
+			(effects
+				(font
+					(size 1.27 1.27)
+				)
+				(justify left)
+			)
+		)
+		(property "Footprint" ""
+			(at 107.442 77.47 90)
+			(effects
+				(font
+					(size 1.27 1.27)
+				)
+				(hide yes)
+			)
+		)
+		(property "Datasheet" "~"
+			(at 109.22 77.47 0)
+			(effects
+				(font
+					(size 1.27 1.27)
+				)
+				(hide yes)
+			)
+		)
+		(property "Description" "Resistor"
+			(at 109.22 77.47 0)
+			(effects
+				(font
+					(size 1.27 1.27)
+				)
+				(hide yes)
+			)
+		)
+		(pin "1"
+		)
+		(pin "2"
+		)
+		(instances
+			(project ""
+				(path "/592a964a-3b7b-4079-9a16-282b0fdb7c03"
+					(reference "R?")
+					(unit 1)
+				)
+			)
+		)
+	)
+	(symbol
 		(lib_id "Device:C_Small")
 		(at 109.22 102.87 90)
@@
 	(symbol
 		(lib_id "Connector:Barrel_Jack_Switch")
-		(at 104.14 74.93 0)
+		(at 91.44 74.93 0)
 		(unit 1)
 		(exclude_from_sim no)
@@
 		(fields_autoplaced yes)
 		(property "Reference" "J1"
-			(at 104.14 66.04 0)
+			(at 91.44 66.04 0)
 			(effects
 				(font
@@
 		)
 		(property "Value" "Barrel_Jack_Switch"
-			(at 104.14 68.58 0)
+			(at 91.44 68.58 0)
 			(effects
 				(font
@@
 		)
 		(property "Footprint" "Connector_BarrelJack:BarrelJack_GCT_DCJ200-10-A_Horizontal"
-			(at 105.41 75.946 0)
+			(at 92.71 75.946 0)
 			(effects
 				(font
@@
 		)
 		(property "Datasheet" "~"
-			(at 105.41 75.946 0)
+			(at 92.71 75.946 0)
 			(effects
 				(font
@@
 		)
 		(property "Description" "DC Barrel Jack with an internal switch"
-			(at 104.14 74.93 0)
+			(at 91.44 74.93 0)
 			(effects
 				(font
@@
 					(unit 1)
 				)
+			)
+		)
+	)
+	(symbol
+		(lib_id "Device:R")
+		(at 102.87 72.39 90)
+		(unit 1)
+		(exclude_from_sim no)
+		(in_bom yes)
+		(on_board yes)
+		(dnp no)
+		(fields_autoplaced yes)
+		(property "Reference" "R?"
+			(at 102.87 66.04 90)
+			(effects
+				(font
+					(size 1.27 1.27)
+				)
+			)
+		)
+		(property "Value" "10k"
+			(at 102.87 68.58 90)
+			(effects
+				(font
+					(size 1.27 1.27)
+				)
+			)
+		)
+		(property "Footprint" ""
+			(at 102.87 74.168 90)
+			(effects
+				(font
+					(size 1.27 1.27)
+				)
+				(hide yes)
+			)
+		)
+		(property "Datasheet" "~"
+			(at 102.87 72.39 0)
+			(effects
+				(font
+					(size 1.27 1.27)
+				)
+				(hide yes)
+			)
+		)
+		(property "Description" "Resistor"
+			(at 102.87 72.39 0)
+			(effects
+				(font
+					(size 1.27 1.27)
+				)
+				(hide yes)
+			)
+		)
+		(pin "1"
+		)
+		(pin "2"
+		)
+		(instances
+			(project ""
+				(path "/592a964a-3b7b-4079-9a16-282b0fdb7c03"
+					(reference "R?")
+					(unit 1)
+				)

Commit message: pcb
Parts:
- removed R?: 12.5k, symbol Device:R
- removed R?: 10k, symbol Device:R
- added R10: 10k, Resistor_SMD:R_0603_1608Metric, symbol Device:R
- added R11: 12.5k, Resistor_SMD:R_0603_1608Metric, symbol Device:R
Connections:
- net GND: now also R11.2
- net at R3.2, R4.1, R9.1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: now also R10.2, R11.1
- net at J1.1: now also R10.1
Changed lines of the file:
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@@
-	)
-	(symbol
-		(lib_id "Device:R")
-		(at 109.22 77.47 0)
-		(unit 1)
-		(exclude_from_sim no)
-		(in_bom yes)
-		(on_board yes)
-		(dnp no)
-		(fields_autoplaced yes)
-		(property "Reference" "R?"
-			(at 111.76 76.1999 0)
-			(effects
-				(font
-					(size 1.27 1.27)
-				)
-				(justify left)
-			)
-		)
-		(property "Value" "12.5k"
-			(at 111.76 78.7399 0)
-			(effects
-				(font
-					(size 1.27 1.27)
-				)
-				(justify left)
-			)
-		)
-		(property "Footprint" ""
-			(at 107.442 77.47 90)
-			(effects
-				(font
-					(size 1.27 1.27)
-				)
-				(hide yes)
-			)
-		)
-		(property "Datasheet" "~"
-			(at 109.22 77.47 0)
-			(effects
-				(font
-					(size 1.27 1.27)
-				)
-				(hide yes)
-			)
-		)
-		(property "Description" "Resistor"
-			(at 109.22 77.47 0)
-			(effects
-				(font
-					(size 1.27 1.27)
-				)
-				(hide yes)
-			)
-		)
-		(pin "1"
-		)
-		(pin "2"
-		)
-		(instances
-			(project ""
-				(path "/592a964a-3b7b-4079-9a16-282b0fdb7c03"
-					(reference "R?")
-					(unit 1)
-				)
-			)
-		)
 	)
 	(symbol
@@
 	)
 	(symbol
+		(lib_id "Device:R")
+		(at 102.87 72.39 90)
+		(unit 1)
+		(exclude_from_sim no)
+		(in_bom yes)
+		(on_board yes)
+		(dnp no)
+		(fields_autoplaced yes)
+		(property "Reference" "R10"
+			(at 102.87 66.04 90)
+			(effects
+				(font
+					(size 1.27 1.27)
+				)
+			)
+		)
+		(property "Value" "10k"
+			(at 102.87 68.58 90)
+			(effects
+				(font
+					(size 1.27 1.27)
+				)
+			)
+		)
+		(property "Footprint" "Resistor_SMD:R_0603_1608Metric"
+			(at 102.87 74.168 90)
+			(effects
+				(font
+					(size 1.27 1.27)
+				)
+				(hide yes)
+			)
+		)
+		(property "Datasheet" "~"
+			(at 102.87 72.39 0)
+			(effects
+				(font
+					(size 1.27 1.27)
+				)
+				(hide yes)
+			)
+		)
+		(property "Description" "Resistor"
+			(at 102.87 72.39 0)
+			(effects
+				(font
+					(size 1.27 1.27)
+				)
+				(hide yes)
+			)
+		)
+		(pin "1"
+		)
+		(pin "2"
+		)
+		(instances
+			(project ""
+				(path "/592a964a-3b7b-4079-9a16-282b0fdb7c03"
+					(reference "R10")
+					(unit 1)
+				)
+			)
+		)
+	)
+	(symbol
+		(lib_id "Device:R")
+		(at 109.22 77.47 0)
+		(unit 1)
+		(exclude_from_sim no)
+		(in_bom yes)
+		(on_board yes)
+		(dnp no)
+		(fields_autoplaced yes)
+		(property "Reference" "R11"
+			(at 111.76 76.1999 0)
+			(effects
+				(font
+					(size 1.27 1.27)
+				)
+				(justify left)
+			)
+		)
+		(property "Value" "12.5k"
+			(at 111.76 78.7399 0)
+			(effects
+				(font
+					(size 1.27 1.27)
+				)
+				(justify left)
+			)
+		)
+		(property "Footprint" "Resistor_SMD:R_0603_1608Metric"
+			(at 107.442 77.47 90)
+			(effects
+				(font
+					(size 1.27 1.27)
+				)
+				(hide yes)
+			)
+		)
+		(property "Datasheet" "~"
+			(at 109.22 77.47 0)
+			(effects
+				(font
+					(size 1.27 1.27)
+				)
+				(hide yes)
+			)
+		)
+		(property "Description" "Resistor"
+			(at 109.22 77.47 0)
+			(effects
+				(font
+					(size 1.27 1.27)
+				)
+				(hide yes)
+			)
+		)
+		(pin "2"
+		)
+		(pin "1"
+		)
+		(instances
+			(project ""
+				(path "/592a964a-3b7b-4079-9a16-282b0fdb7c03"
+					(reference "R11")
+					(unit 1)
+				)
+			)
+		)
+	)
+	(symbol
 		(lib_id "Device:LED")
 		(at 181.61 87.63 180)
@@
 					(unit 1)
 				)
-			)
-		)
-	)
-	(symbol
-		(lib_id "Device:R")
-		(at 102.87 72.39 90)
-		(unit 1)
-		(exclude_from_sim no)
-		(in_bom yes)
-		(on_board yes)
-		(dnp no)
-		(fields_autoplaced yes)
-		(property "Reference" "R?"
-			(at 102.87 66.04 90)
-			(effects
-				(font
-					(size 1.27 1.27)
-				)
-			)
-		)
-		(property "Value" "10k"
-			(at 102.87 68.58 90)
-			(effects
-				(font
-					(size 1.27 1.27)
-				)
-			)
-		)
-		(property "Footprint" ""
-			(at 102.87 74.168 90)
-			(effects
-				(font
-					(size 1.27 1.27)
-				)
-				(hide yes)
-			)
-		)
-		(property "Datasheet" "~"
-			(at 102.87 72.39 0)
-			(effects
-				(font
-					(size 1.27 1.27)
-				)
-				(hide yes)
-			)
-		)
-		(property "Description" "Resistor"
-			(at 102.87 72.39 0)
-			(effects
-				(font
-					(size 1.27 1.27)
-				)
-				(hide yes)
-			)
-		)
-		(pin "1"
-		)
-		(pin "2"
-		)
-		(instances
-			(project ""
-				(path "/592a964a-3b7b-4079-9a16-282b0fdb7c03"
-					(reference "R?")
-					(unit 1)
-				)

Commit message: updated schematic
Parts:
- removed R10: 10k, Resistor_SMD:R_0603_1608Metric, symbol Device:R
- removed R11: 12.5k, Resistor_SMD:R_0603_1608Metric, symbol Device:R
- added C3, C4: 10u, Capacitor_SMD:C_0603_1608Metric, symbol Device:C_Small
- added R7: 1.6k, Resistor_SMD:R_0603_1608Metric, symbol Device:R
- added R8: 4.7k, Resistor_SMD:R_0603_1608Metric, symbol Device:R
- added U2: LM7805_TO220, Package_TO_SOT_THT:TO-220-3_Vertical, symbol Regulator_Linear:LM7805_TO220
- renumbered R2 to R1, R8 to R10, R9 to R11, R1 to R2, R7 to R9
Connections:
- net GND: now also C3.2, C4.2, R8.1
- net at J1.1: now also C3.1, U2.1 (VI)
- net +5V: now reaches R11.1, R3.2, R4.1, U1.4 (V+)
- net +5V: now also C4.1, R7.1, U2.3 (VO)
- new net: R7.2, R8.2, U2.2 (GND)
Other:
- moved on the sheet: J1

Commit message: changes to pcb
Parts:
- C1, C2, C3, C4: footprint Capacitor_SMD:C_0603_1608Metric -> Capacitor_SMD:C_0805_2012Metric
- R1, R10, R11, R2, R3, R4, R5, R6, R7, R8, R9: footprint Resistor_SMD:R_0603_1608Metric -> Resistor_SMD:R_0805_2012Metric
Changed lines of the file:
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@@
 			)
 		)
-		(property "Footprint" "Resistor_SMD:R_0603_1608Metric"
+		(property "Footprint" "Resistor_SMD:R_0805_2012Metric"
 			(at 109.22 98.298 90)
 			(effects
@@
 			)
 		)
-		(property "Footprint" "Capacitor_SMD:C_0603_1608Metric"
+		(property "Footprint" "Capacitor_SMD:C_0805_2012Metric"
 			(at 109.22 102.87 0)
 			(effects
@@
 			)
 		)
-		(property "Footprint" "Capacitor_SMD:C_0603_1608Metric"
+		(property "Footprint" "Capacitor_SMD:C_0805_2012Metric"
 			(at 132.08 40.64 0)
 			(effects
@@
 			)
 		)
-		(property "Footprint" "Resistor_SMD:R_0603_1608Metric"
+		(property "Footprint" "Resistor_SMD:R_0805_2012Metric"
 			(at 172.72 103.378 90)
 			(effects
@@
 			)
 		)
-		(property "Footprint" "Resistor_SMD:R_0603_1608Metric"
+		(property "Footprint" "Resistor_SMD:R_0805_2012Metric"
 			(at 156.718 52.07 90)
 			(effects
@@
 			)
 		)
-		(property "Footprint" "Resistor_SMD:R_0603_1608Metric"
+		(property "Footprint" "Resistor_SMD:R_0805_2012Metric"
 			(at 153.162 41.91 90)
 			(effects
@@
 			)
 		)
-		(property "Footprint" "Resistor_SMD:R_0603_1608Metric"
+		(property "Footprint" "Resistor_SMD:R_0805_2012Metric"
 			(at 118.618 86.36 90)
 			(effects
@@
 			)
 		)
-		(property "Footprint" "Resistor_SMD:R_0603_1608Metric"
+		(property "Footprint" "Resistor_SMD:R_0805_2012Metric"
 			(at 172.72 114.808 90)
 			(effects
@@
 			)
 		)
-		(property "Footprint" "Resistor_SMD:R_0603_1608Metric"
+		(property "Footprint" "Resistor_SMD:R_0805_2012Metric"
 			(at 141.478 92.71 90)
 			(effects
@@
 			)
 		)
-		(property "Footprint" "Capacitor_SMD:C_0603_1608Metric"
+		(property "Footprint" "Capacitor_SMD:C_0805_2012Metric"
 			(at 107.95 119.38 0)
 			(effects
@@
 			)
 		)
-		(property "Footprint" "Resistor_SMD:R_0603_1608Metric"
+		(property "Footprint" "Resistor_SMD:R_0805_2012Metric"
 			(at 172.72 89.408 90)
 			(effects
@@
 			)
 		)
-		(property "Footprint" "Capacitor_SMD:C_0603_1608Metric"
+		(property "Footprint" "Capacitor_SMD:C_0805_2012Metric"
 			(at 165.1 40.64 0)
 			(effects
@@
 			)
 		)
-		(property "Footprint" "Resistor_SMD:R_0603_1608Metric"
+		(property "Footprint" "Resistor_SMD:R_0805_2012Metric"
 			(at 141.478 104.14 90)
 			(effects
@@
 			)
 		)
-		(property "Footprint" "Resistor_SMD:R_0603_1608Metric"
+		(property "Footprint" "Resistor_SMD:R_0805_2012Metric"
 			(at 137.922 78.74 90)
 			(effects
@@
 			)
 		)
-		(property "Footprint" "Resistor_SMD:R_0603_1608Metric"
+		(property "Footprint" "Resistor_SMD:R_0805_2012Metric"
 			(at 111.252 119.38 90)
 			(effects

Commit message: comments and schematic update
Parts:
- added C5: 100n, Capacitor_SMD:C_0805_2012Metric, symbol Device:C_Small
- renumbered C3 to C1, C4 to C2, C1 to C3, C2 to C4, R7 to R1, R8 to R2, R1 to R3, R2 to R4, R3 to R5, R4 to R6, R5 to R7, R6 to R8, U2 to U1, U1 to U2
Connections:
- net +5V: now also C5.1
- net GND: now also C5.2
Other:
- moved on the sheet: C1, C2, J1, R1, R2, U1, U2E
