File: analog/kicad/scheme.kicad_pcb (KiCad board)
At the start: 2 copper layers, 62.5 x 27 mm, 25 parts, among them J1 Barrel_Jack_Switch, U1 LM7805_TO220, U2 LM324

Commit message: remove text
Other:
- board text removed: "Peale vaadates on trükkplaat üsna kena, aga mõned asjad jäid silma 1) Komponentide nimed R5, R6 ja D4 on kindlasti liiga trükkplaadi ääre lähedal 2) Mõelge kindlasti, kas saate 0603 komponentide jootmisega hakkama 3) Hetkel on trükkplaadi rajad 0.2 mm ehk ac 8 milsi laiad. ise soovitan rajad teha kindlasti 10/10 reeglite järgi, kusjuures toite rajad soovitan teha isegi laiemad, kuni 40 mils. Kuna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"
Changed lines of the file:
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@@
 		(layer "Edge.Cuts")
-	)
-	(gr_text "Peale vaadates on trükkplaat üsna kena, aga mõned asjad jäid silma\n1) Komponentide nimed R5, R6 ja D4 on kindlasti liiga trükkplaadi ääre lähedal\n2) Mõelge kindlasti, kas saate 0603 komponentide jootmisega hakkama\n3) Hetkel on trükkplaadi rajad 0.2 mm ehk ac 8 milsi laiad. ise soovitan rajad teha kindlasti 10/10\nreeglite järgi, kusjuures toite rajad soovitan teha isegi laiemad, kuni 40 mils. \nKuna plaadil ruumi on, siis ega paha ei tee, kui ka muud rajad on laiemad\n4) lisage nn Power good LED (ehk toitesse üks, mis lihtaslt indikeerib, kas toide on olemas või ei)\n5) Soovitan mõelda, et kas trükkplaat läheb ka kusagile korpusesse ja siis teha \ntrükkplaadi väliskuju korpuse järgi\n6) Viade suurus on hetkel 03/06, soovitan vähemalt 05/08 suurust\n7) Võite kaaluda ka valgusdioodide SMD vastu vahetamisele (aga see on teie otsus).\nKui seade läheb nt korpusesse, ehk ongi THT komponent parem).\n8) U1 on ka kindlasti SMD-na saadaval. Kaaluge, kas selle kasutamine võiks anda mingisuguseid eeliseid\n9) Skeemis vististi mainisin, aga U1 tahab kindlasti toitekondensaatorit ning sisend tahab kaitsmist\n10) Paigutuse mõistes mõelge sellele, et kuivõrd D2-D4 võivad hakata mõjutama mõõtetulemusi. Ehk on kasulikum D2-D4\npaigutada nii, et nad saab plaadiga tasapinda panna (hetkel 90 kraadise nurga all)\n11) Ehk on toite osas mõistlik mõelda mingisuguse patarei lahenduse peale (+ siis sisse/väljalülitamiseks\nmingisugune lüliti ka)\n"
-		(at 107.6 127.8 0)
-		(layer "F.Cu")
-		(effects
-			(font
-				(size 1.27 1.27)
-			)
-			(justify left)
-		)
 	)
 	(segment

Commit message: pcb changes
Parts:
- removed J1: Barrel_Jack_Switch, Connector_BarrelJack:BarrelJack_GCT_DCJ200-10-A_Horizontal
- removed the R7 at (131.4, 95.0)
- removed the R8 at (131.4, 90.8)
- added BT1: Battery_Cell 9V, Battery:BatteryHolder_Eagle_12BH611-GR, B.Cu at (108.6, 98.4)
- added D6: SMAJ13A, Diode_SMD:D_SMA, F.Cu at (86.5, 79.9)
- added F1: SMDH1206B005TF, Resistor_SMD:R_1206_3216Metric, F.Cu at (85.0, 84.0)
- added SW1: SW_Nidec_CAS-120A1, Button_Switch_SMD:Nidec_Copal_CAS-120A, F.Cu at (91.2, 92.0)
- U2: footprint Package_DIP:DIP-14_W7.62mm_Socket -> Package_DIP:DIP-14_W7.62mm_SMDSocket_SmallPads
- moved C4 54.3 mm to (83.5, 106.2), turned to -90 degrees
- moved U1 46.3 mm to (83.5, 89.5), turned to -90 degrees
- moved R10 43.7 mm to (88.8, 106.2), turned to -90 degrees
- moved C3 41.5 mm to (87.0, 100.0), turned to 180 degrees
- moved D1 36.4 mm to (99.0, 89.5), turned to -90 degrees
- moved D5 36.4 mm to (93.4, 106.2), turned to -90 degrees
- moved C1 35.6 mm to (105.2, 91.9), turned to 90 degrees
- moved R2 29.0 mm to (108.6, 91.9), turned to 90 degrees
- moved R6 25.9 mm to (139.9, 83.9)
- moved C5 25.7 mm to (110.8, 103.5), turned to -90 degrees
- moved R5 25.1 mm to (133.9, 83.9)
- moved R1 23.2 mm to (119.3, 92.3), turned to 180 degrees
- moved C2 21.4 mm to (119.3, 95.7), turned to 180 degrees
- moved U2 16.4 mm to (132.6, 91.8), turned to 90 degrees
- moved R3 16.4 mm to (124.1, 99.7), turned to 90 degrees
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- renumbered R12 to R10, R9 to R7, R10 to R8, R11 to R9
Connections:
- net /OUT renamed TIA_OUT
- net /dist2 renamed /(1.7V)
- net /dist3 renamed (2.5V)
- C2 pad 1: GND -> VGND
- C2 pad 2: /BIAS -> GND
- C3 pad 1: Net-(U1-VI) -> Net-(SW1-A)
- R1 pad 1: GND -> VGND
- R1 pad 2: /BIAS -> GND
- R3 pad 1: /BIAS -> +5V
- R3 pad 2: +5V -> VGND
- U1 pad 1: Net-(U1-VI) -> Net-(D6-A1)
- U1 pad 2: Net-(U1-GND) -> GND
- U2 pad 3: /BIAS -> VGND
Routing:
- net Net-(BT1-+): track 0.00 -> 20.6 mm
- net (2.5V): track 21.8 -> 41.6 mm, vias 0 -> 2
- net Net-(SW1-A): track 0.00 -> 18.3 mm
- net /BIAS: track 17.3 -> 0.00 mm, vias 1 -> 0
- net VGND: track 0.00 -> 15.8 mm
- net Net-(D1-A): track 16.1 -> 31.9 mm, vias 1 -> 2
- net +5V: track 95.1 -> 109.1 mm, vias 4 -> 0
- net TIA_OUT: track 29.2 -> 42.7 mm
- net Net-(R8-Pad1): track 10.1 -> 22.2 mm
- net Net-(U1-VI): track 11.5 -> 0.00 mm
- net Net-(U1-GND): track 10.4 -> 0.00 mm
- net Net-(D6-A1): track 0.00 -> 9.96 mm
- net Net-(R7-Pad1): track 26.3 -> 21.9 mm, vias 2 -> 0
- net /(1.7V): track 11.8 -> 9.45 mm
- net Net-(D2-A): track 3.63 -> 5.04 mm
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Other:
- board size 62.5 x 27 mm -> 91 x 34.3 mm

Commit message: more analog cleanup
Parts:
- moved C1 82.7 mm to (45.6, 34.5)
- moved D5 82.7 mm to (33.8, 48.8)
- moved BT1 82.7 mm to (49.0, 41.0)
- moved C2 82.7 mm to (59.7, 38.3)
- moved C3 82.7 mm to (27.4, 42.6)
- moved C4 82.7 mm to (24.0, 48.8)
- moved C5 82.7 mm to (51.2, 46.0)
- moved D2 82.7 mm to (107.4, 33.3)
- moved D3 82.7 mm to (107.4, 25.1)
- moved D4 82.7 mm to (107.4, 41.4)
- moved D6 82.7 mm to (26.9, 22.5)
- moved F1 82.7 mm to (25.4, 26.6)
- moved R10 82.7 mm to (29.2, 48.8)
- moved R2 82.7 mm to (49.0, 34.5)
- moved R3 82.7 mm to (64.5, 42.3)
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
Commit message: pcb changes
Parts:
- D2, D3, D4: footprint LED_THT:LED_D5.0mm -> LED_THT:LED_D5.0mm_Horizontal_O1.27mm_Z3.0mm; moved to B.Cu
- D5, U1: moved to B.Cu
- moved D5 2.66 mm to (36.5, 48.8)
- moved C3 2.06 mm to (29.5, 42.6), turned to 0 degrees
- moved D4 0.19 mm to (107.5, 41.2)
- moved D3 0.13 mm to (107.5, 25.2)
- moved D2 0.09 mm to (107.5, 33.2)
Routing:
- net Net-(D5-A): track 4.61 -> 7.28 mm, vias 0 -> 1
